File: Power Supply.kicad_sch (KiCad schematic)
At the start: 30 parts, among them SW1 SW_SPDT, U1 LM7812_TO220, U2 LM7912_TO220, U3 LM7805_TO220

Commit message: Finish schematic
Parts:
- removed C10, C9: 1u, Capacitor_THT:C_Disc_D5.0mm_W2.5mm_P5.00mm, symbol Device:C
- removed D10, D9: 1N5819, Diode_THT:D_DO-41_SOD81_P10.16mm_Horizontal, symbol Diode:1N5819
- removed D11: LED, LED_THT:LED_D5.0mm, symbol Device:LED
- removed R3: 22k, Resistor_THT:R_Axial_DIN0207_L6.3mm_D2.5mm_P7.62mm_Horizontal, symbol Device:R
- removed U3: LM7805_TO220, Package_TO_SOT_THT:TO-220-3_Vertical, symbol Regulator_Linear:LM7805_TO220
- SW201: renamed from SW1; footprint Switch:MTS-102_MTS-103_MTS-112_MTS-113_MTS-123 -> Custom:MTS-102_MTS-103_MTS-112_MTS-113_MTS-123
- renumbered C1 to C201, C2 to C202, C3 to C203, C4 to C204, C5 to C205, C6 to C206, C7 to C207, C8 to C208, D1 to D201, D2 to D202, D3 to D203, D4 to D204, D5 to D205, D6 to D206, D7 to D207, D8 to D208, H1 to H201, H2 to H202, R1 to R201, R2 to R202, U1 to U201, U2 to U202
Other:
- moved on the sheet: C201, C202, C203, C204, C205, C206, C207, C208, D201, D202, D203, D204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
