File: White Noise.kicad_sch (KiCad schematic)
At the start: 17 parts

Commit message: Finish schematic
Parts:
- removed RV?: 50k, Potentiometer_THT:Potentiometer_Alpha_RD901F-40-00D_Single_Vertical_CircularHoles, symbol Device:R_Potentiometer
- added R2007: 47k, Resistor_THT:R_Axial_DIN0207_L6.3mm_D2.5mm_P7.62mm_Horizontal, symbol Device:R
- gave numbers to parts that had none: 14
Connections:
- net +12V: no longer U2001.8 (V+)
- net -12V: no longer U2001.4 (V-)
- net OUT: now also U2001.1, R2007.2; no longer U2001.7
- net at R2006.1: now also U2001.2 (-), R2007.1; no longer U2001.6 (-)
- net at R2005.2, U2001.1: now also U2001.3 (+); no longer U2001.5 (+)
