File: SD.kicad_sch (KiCad schematic)
At the start: 31 parts, among them J2201 AudioJack2_SwitchT, J2202 AudioJack2_SwitchT, J2203 AudioJack2_SwitchT, J2204 AudioJack2_SwitchT, J2205 AudioJack2_SwitchT, U2201 TL072

Commit message: Update VCO
Parts:
- removed C2201: 1n, Capacitor_THT:C_Disc_D5.0mm_W2.5mm_P5.00mm, symbol Device:C
- renumbered C2202 to C2201, C2203 to C2202, C2204 to C2203
Connections:
- net -12V: now also RV2203.3
- net GND: no longer RV2203.3
Other:
- sheet VCO ports: added none; removed TIMING_CAP_1, TIMING_CAP_2
Changed lines of the file:
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@@
-    (stroke (width 0) (type default) (color 0 0 0 0))
-  )
-  (wire (pts (xy 64.77 105.41) (xy 63.5 105.41))
     (stroke (width 0) (type default) (color 0 0 0 0))
   )
@@
     (stroke (width 0) (type default) (color 0 0 0 0))
   )
-  (wire (pts (xy 60.96 101.6) (xy 60.96 124.46))
-    (stroke (width 0) (type default) (color 0 0 0 0))
-  )
   (wire (pts (xy 214.63 53.34) (xy 218.44 53.34))
     (stroke (width 0) (type default) (color 0 0 0 0))
@@
     (stroke (width 0) (type default) (color 0 0 0 0))
   )
-  (wire (pts (xy 63.5 105.41) (xy 63.5 113.03))
-    (stroke (width 0) (type default) (color 0 0 0 0))
-  )
   (wire (pts (xy 92.71 46.99) (xy 92.71 29.21))
     (stroke (width 0) (type default) (color 0 0 0 0))
@@
     (stroke (width 0) (type default) (color 0 0 0 0))
   )
-  (wire (pts (xy 78.74 124.46) (xy 78.74 113.03))
-    (stroke (width 0) (type default) (color 0 0 0 0))
-  )
   (wire (pts (xy 209.55 120.65) (xy 203.2 120.65))
     (stroke (width 0) (type default) (color 0 0 0 0))
@@
     (stroke (width 0) (type default) (color 0 0 0 0))
   )
-  (wire (pts (xy 64.77 101.6) (xy 60.96 101.6))
-    (stroke (width 0) (type default) (color 0 0 0 0))
-  )
   (wire (pts (xy 226.06 102.87) (xy 226.06 85.09))
     (stroke (width 0) (type default) (color 0 0 0 0))
@@
     (stroke (width 0) (type default) (color 0 0 0 0))
   )
-  (wire (pts (xy 60.96 124.46) (xy 71.12 124.46))
-    (stroke (width 0) (type default) (color 0 0 0 0))
-  )
   (wire (pts (xy 121.92 53.34) (xy 125.73 53.34))
     (stroke (width 0) (type default) (color 0 0 0 0))
   )
   (wire (pts (xy 226.06 106.68) (xy 228.6 106.68))
-    (stroke (width 0) (type default) (color 0 0 0 0))
-  )
-  (wire (pts (xy 78.74 113.03) (xy 63.5 113.03))
     (stroke (width 0) (type default) (color 0 0 0 0))
   )
@@
     (pin "3")
   )
-  (symbol (lib_id "power:GND") (at 50.8 97.79 0) (unit 1)
-    (in_bom yes) (on_board yes) (fields_autoplaced)
-    (property "Reference" "#PWR02206" (id 0) (at 50.8 104.14 0)
-      (effects (font (size 1.27 1.27)) hide)
-    )
-    (property "Value" "GND" (id 1) (at 50.8 102.87 0))
-    (property "Footprint" "" (id 2) (at 50.8 97.79 0)
-      (effects (font (size 1.27 1.27)) hide)
-    )
-    (property "Datasheet" "" (id 3) (at 50.8 97.79 0)
-      (effects (font (size 1.27 1.27)) hide)
-    )
-    (pin "1")
-  )
   (symbol (lib_id "Device:R_Potentiometer") (at 50.8 93.98 0) (unit 1)
     (in_bom yes) (on_board yes) (fields_autoplaced)
@@
   (symbol (lib_id "Device:C") (at 168.91 138.43 90) (unit 1)
     (in_bom yes) (on_board yes)
-    (property "Reference" "C2202" (id 0) (at 168.91 132.0292 90))
+    (property "Reference" "C2201" (id 0) (at 168.91 132.0292 90))
     (property "Value" "0.1u" (id 1) (at 168.91 134.3406 90))
     (property "Footprint" "Capacitor_THT:C_Disc_D5.0mm_W2.5mm_P5.00mm" (id 2) (at 172.72 137.4648 0)
@@
     (pin "1")
   )
-  (symbol (lib_id "Device:C") (at 74.93 124.46 270) (unit 1)
-    (in_bom yes) (on_board yes) (fields_autoplaced)
-    (property "Reference" "C2201" (id 0) (at 74.93 116.84 90))
-    (property "Value" "1n" (id 1) (at 74.93 119.38 90))
-    (property "Footprint" "Capacitor_THT:C_Disc_D5.0mm_W2.5mm_P5.00mm" (id 2) (at 71.12 125.4252 0)
-      (effects (font (size 1.27 1.27)) hide)
-    )
-    (property "Datasheet" "~" (id 3) (at 74.93 124.46 0)
-      (effects (font (size 1.27 1.27)) hide)
-    )
-    (pin "1")
-    (pin "2")
-  )
   (symbol (lib_id "power:-12V") (at 50.8 165.1 180) (unit 1)
     (in_bom yes) (on_board yes) (fields_autoplaced)
@@
   (symbol (lib_id "Device:C") (at 196.85 99.06 90) (unit 1)
     (in_bom yes) (on_board yes) (fields_autoplaced)
-    (property "Reference" "C2204" (id 0) (at 196.85 91.44 90))
+    (property "Reference" "C2203" (id 0) (at 196.85 91.44 90))
     (property "Value" "0.1u" (id 1) (at 196.85 93.98 90))
     (property "Footprint" "Capacitor_THT:C_Disc_D5.0mm_W2.5mm_P5.00mm" (id 2) (at 200.66 98.0948 0)
@@
     (pin "1")
   )
+  (symbol (lib_id "power:-12V") (at 50.8 97.79 180) (unit 1)
+    (in_bom yes) (on_board yes) (fields_autoplaced)
+    (property "Reference" "#PWR02206" (id 0) (at 50.8 100.33 0)
+      (effects (font (size 1.27 1.27)) hide)
+    )
+    (property "Value" "-12V" (id 1) (at 50.8 102.87 0))
+    (property "Footprint" "" (id 2) (at 50.8 97.79 0)
+      (effects (font (size 1.27 1.27)) hide)
+    )
+    (property "Datasheet" "" (id 3) (at 50.8 97.79 0)
+      (effects (font (size 1.27 1.27)) hide)
+    )
+    (pin "1")
+  )
   (symbol (lib_id "Connector:AudioJack2_SwitchT") (at 30.48 105.41 0) (mirror x) (unit 1)
     (in_bom yes) (on_board yes) (fields_autoplaced)
@@
   (symbol (lib_id "Device:C") (at 168.91 153.67 90) (unit 1)
     (in_bom yes) (on_board yes)
-    (property "Reference" "C2203" (id 0) (at 168.91 147.2692 90))
+    (property "Reference" "C2202" (id 0) (at 168.91 147.2692 90))
     (property "Value" "0.1u" (id 1) (at 168.91 149.5806 90))
     (property "Footprint" "Capacitor_THT:C_Disc_D5.0mm_W2.5mm_P5.00mm" (id 2) (at 172.72 152.7048 0)
@@
     )
   )
-  (sheet (at 64.77 87.63) (size 20.32 20.32) (fields_autoplaced)
+  (sheet (at 64.77 87.63) (size 20.32 12.7) (fields_autoplaced)
     (stroke (width 0.1524) (type solid) (color 0 0 0 0))
     (fill (color 0 0 0 0.0000))
@@
       (effects (font (size 1.27 1.27)) (justify left bottom))
     )
-    (property "Sheet file" "VCO.kicad_sch" (id 1) (at 64.77 108.5346 0)
+    (property "Sheet file" "VCO.kicad_sch" (id 1) (at 64.77 100.9146 0)
       (effects (font (size 1.27 1.27)) (justify left top))
     )
@@
       (effects (font (size 1.27 1.27)) (justify left))
     )
-    (pin "TIMING_CAP_1" bidirectional (at 64.77 101.6 180)
-      (effects (font (size 1.27 1.27)) (justify left))
-    )
-    (pin "TIMING_CAP_2" bidirectional (at 64.77 105.41 180)
-      (effects (font (size 1.27 1.27)) (justify left))
-    )
