File: HPF.kicad_sch (KiCad schematic)
At the start: 41 parts, among them Q2101 BC558, Q2102 BC558, U2101 TL072, U2102 TL072, U2103 CA3080, U2104 CA3080

Commit message: Finish PCB
Parts:
- renumbered R2103 to R2104, R2104 to R2105, R2105 to R2106, R2106 to R2107, R2107 to R2108, R2108 to R2109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
Connections:
- net at C2101.1, U2101.2 (-): now also Q2101.1 (C), R2105.1
