File: Panel/Panel.kicad_pcb (KiCad board)
At the start: 2 copper layers, 271.7 x 266.7 mm, 0 parts

Commit message: Resize panel
Routing:
- added copper zone on B.Cu, net (none)
- added copper zone on F.Cu, net (none)
Other:
- board size 271.7 x 266.7 mm -> 333 x 387.6 mm
